Commit message: new approach to fix rviz display of robot

File: writing_robot_description/urdf/robot_arm.urdf (robot description, URDF)
Before this commit: robot writing_arm, 6 links, 5 joints
Links:
- removed link link_1
- removed link link_2
- removed link link_3
- added link forearm_link, mass 0.15; visual mesh filename=package://writing_robot_description/meshes/Follower_Elbow_T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 scale=0.001 0.001 0.001; visual mesh filename=package://writing_robot_description/meshes/XL,XC-330.stl scale=0.001 0.001 0.001
- added link hand_link, mass 0.08; visual mesh filename=package://writing_robot_description/meshes/Follower_Elbow_T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 scale=0.001 0.001 0.001; visual mesh filename=package://writing_robot_description/meshes/XL,XC-330.stl scale=0.001 0.001 0.001
- added link shoulder_link, mass 0.3; visual mesh filename=package://writing_robot_description/meshes/XL-430_new.stl scale=0.001 0.001 0.001; visual mesh filename=package://writing_robot_description/meshes/fr12_s102.stl scale=0.001 0.001 0.001
- added link upper_arm_link, mass 0.2; visual mesh filename=package://writing_robot_description/meshes/Follower_Shoulde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 scale=0.001 0.001 0.001; visual mesh filename=package://writing_robot_description/meshes/XL,XC-330.stl scale=0.001 0.001 0.001
- added link wrist_link, mass 0.1; visual mesh filename=package://writing_robot_description/meshes/Follower_Elbow_T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 scale=0.001 0.001 0.001; visual mesh filename=package://writing_robot_description/meshes/XL,XC-330.stl scale=0.001 0.001 0.001
- link base_link: mass None -> 0.5; geometry collision cylinder length=0.02 radius=0.05; visual mesh filename=package://writing_robot_description/meshes/Follower_Base_bi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 scale=0.001 0.001 0.001
- link pen_link: mass None -> 0.02; geometry visual mesh filename=package://writing_robot_description/meshes/Follower_Gripper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 scale=0.001 0.001 0.001; visual mesh filename=package://writing_robot_description/meshes/XL,XC-330.stl scale=0.001 0.001 0.001
- link pen_tip: geometry visual mesh filename=package://writing_robot_description/meshes/Follower_Gripper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 scale=0.001 0.001 0.001
Joints:
- removed joint joint_1
- removed joint joint_2
- removed joint joint_3
- removed joint joint_4
- added joint elbow_flex: type revolute, parent upper_arm_link, child forearm_link, origin xyz=0.111000 -0.007000 -0.113000 rpy=1.570796 -1.570796 0.000000, axis 0.000000 -1.000000 0.000000, limit lower=-2.5 upper=2.5 effort=1.5 velocity=3.14
- added joint pen_holder: type revolute, parent hand_link, child pen_link, origin xyz=-0.055000 0.008000 0.213000 rpy=3.141593 0.000000 1.570796, axis 0.000000 0.000000 1.000000, limit lower=-0.5 upper=0.5 effort=0.5 velocity=1.57
- added joint shoulder_lift: type revolute, parent shoulder_link, child upper_arm_link, origin xyz=0.000000 0.002000 -0.001000 rpy=1.570796 1.570796 -1.570796, axis 1.000000 0.000000 0.000000, limit lower=-2.0 upper=2.0 effort=2.0 velocity=3.14
- added joint shoulder_pan: type revolute, parent base_link, child shoulder_link, origin xyz=0.000000 0.000000 0.059000 rpy=1.570796 0.000000 0.000000, axis 0.000000 -1.000000 0.000000, limit lower=-3.14159 upper=3.14159 effort=2.0 velocity=3.14
- added joint wrist_flex: type revolute, parent forearm_link, child wrist_link, origin xyz=0.000000 0.038000 -0.021000 rpy=1.570796 -0.000000 0.000000, axis 0.000000 0.000000 -1.000000, limit lower=-2.0 upper=2.0 effort=1.5 velocity=3.14
- added joint wrist_roll: type revolute, parent wrist_link, child hand_link, origin xyz=0.008000 0.009000 0.019000 rpy=0.000000 1.570796 0.000000, axis -1.000000 0.000000 0.000000, limit lower=-3.14159 upper=3.14159 effort=1.0 velocity=3.14
- joint pen_tip_joint: origin xyz=0.10 0 0 rpy=0 0 0 -> xyz=0.05 0 0 rpy=0 0 0

Commit message: intermediate changes

File: writing_robot_description/urdf/robot_arm.urdf (robot description, URDF)
Before this commit: robot koch_v11_writing_arm, 8 links, 7 joints
Joints:
- joint elbow_flex: axis 0.000000 -1.000000 0.000000 -> 0.000000 0.000000 -1.000000; origin xyz=0.111000 -0.007000 -0.113000 rpy=1.570796 -1.570796 0.000000 -> xyz=0.014000 -0.137000 0.003000 rpy=-1.570796 1.570796 0.000000

Commit message: elbow flex fixed in display

File: writing_robot_description/urdf/robot_arm.urdf (robot description, URDF)
Before this commit: robot koch_v11_writing_arm, 8 links, 7 joints
Joints:
- joint elbow_flex: axis 0.000000 0.000000 -1.000000 -> 1.000000 0.000000 0.000000; origin xyz=0.014000 -0.137000 0.003000 rpy=-1.570796 1.570796 0.000000 -> xyz=-0.000000 -0.108000 0.014000 rpy=0.000000 -0.000000 -0.000000

Commit message: hand link donegit add writing_robot_description/urdf/robot_arm.urdf

File: writing_robot_description/urdf/robot_arm.urdf (robot description, URDF)
Before this commit: robot koch_v11_writing_arm, 8 links, 7 joints
Links:
- removed link pen_tip
- link hand_link: geometry visual mesh filename=package://writing_robot_description/meshes/Follower_Gripper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 scale=0.001 0.001 0.001; visual mesh filename=package://writing_robot_description/meshes/XL,XC-330.stl scale=0.001 0.001 0.001
- link pen_link: geometry visual mesh filename=package://writing_robot_description/meshes/Follower_Gripper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 scale=0.001 0.001 0.001
Joints:
- removed joint pen_tip_joint
- joint pen_holder: axis 0.000000 0.000000 1.000000 -> 0.000000 -1.000000 0.000000; origin xyz=-0.055000 0.008000 0.213000 rpy=3.141593 0.000000 1.570796 -> xyz=-0.342000 0.011000 -0.205000 rpy=0.000000 0.000000 0.000000
- joint wrist_flex: axis 0.000000 0.000000 -1.000000 -> -1.000000 0.000000 0.000000; origin xyz=0.000000 0.038000 -0.021000 rpy=1.570796 -0.000000 0.000000 -> xyz=-0.001000 -0.100000 0.002000 rpy=0.000000 -0.000000 -0.000000
- joint wrist_roll: axis -1.000000 0.000000 0.000000 -> 0.000000 0.000000 1.000000; origin xyz=0.008000 0.009000 0.019000 rpy=0.000000 1.570796 0.000000 -> xyz=0.003000 -0.001000 -0.044000 rpy=3.141593 -0.000000 -1.570796

Commit message: pen_link working

File: writing_robot_description/urdf/robot_arm.urdf (robot description, URDF)
Before this commit: robot koch_v11_writing_arm, 7 links, 6 joints
Joints:
- joint pen_holder: axis 0.000000 -1.000000 0.000000 -> 0.000000 1.000000 0.000000; origin xyz=-0.342000 0.011000 -0.205000 rpy=0.000000 0.000000 0.000000 -> xyz=0.000000 -0.009000 0.015000 rpy=0.000000 -0.000000 -1.570796

Commit message: next try

File: writing_robot_description/urdf/robot_arm.urdf (robot description, URDF)
Before this commit: robot koch_v11_writing_arm, 7 links, 6 joints
Joints:
- joint elbow_flex: origin xyz=-0.000000 -0.108000 0.014000 rpy=0.000000 -0.000000 -0.000000 -> xyz=0.109000 0.000000 -0.014000 rpy=0.000000 0.000000 0.000000
- joint pen_holder: origin xyz=0.000000 -0.009000 0.015000 rpy=0.000000 -0.000000 -1.570796 -> xyz=-0.001000 -0.008000 0.015000 rpy=0.000000 0.000000 0.000000
- joint shoulder_lift: origin xyz=0.000000 0.002000 -0.001000 rpy=1.570796 1.570796 -1.570796 -> xyz=-0.001000 0.000000 0.038000 rpy=0.000000 0.000000 0.000000
- joint shoulder_pan: origin xyz=0.000000 0.000000 0.059000 rpy=1.570796 0.000000 0.000000 -> xyz=0.001000 0.000000 0.021000 rpy=0.000000 0.000000 0.000000
- joint wrist_flex: axis -1.000000 0.000000 0.000000 -> 1.000000 0.000000 0.000000; origin xyz=-0.001000 -0.100000 0.002000 rpy=0.000000 -0.000000 -0.000000 -> xyz=0.101000 0.000000 0.002000 rpy=0.000000 0.000000 0.000000
- joint wrist_roll: origin xyz=0.003000 -0.001000 -0.044000 rpy=3.141593 -0.000000 -1.570796 -> xyz=-0.001000 0.000000 0.039000 rpy=0.000000 0.000000 0.000000

Commit message: axis change

File: writing_robot_description/urdf/robot_arm.urdf (robot description, URDF)
Before this commit: robot koch_v11_writing_arm, 7 links, 6 joints
Joints:
- joint elbow_flex: axis 1.000000 0.000000 0.000000 -> 0.000000 1.000000 0.000000
- joint pen_holder: axis 0.000000 1.000000 0.000000 -> -1.000000 0.000000 0.000000
- joint shoulder_lift: axis 1.000000 0.000000 0.000000 -> 0.000000 1.000000 0.000000
- joint shoulder_pan: axis 0.000000 -1.000000 0.000000 -> 0.000000 0.000000 1.000000
- joint wrist_flex: axis 1.000000 0.000000 0.000000 -> 0.000000 1.000000 0.000000

Commit message: fixed thumb

File: writing_robot_description/urdf/robot_arm.urdf (robot description, URDF)
Before this commit: robot koch_v11_writing_arm, 7 links, 6 joints
Joints:
- joint pen_holder: origin xyz=-0.001000 -0.008000 0.015000 rpy=0.000000 0.000000 0.000000 -> xyz=0.000000 -0.007000 0.015000 rpy=0.000000 0.000000 0.000000

Commit message: reflect latest real robot urdf to display-only version

File: writing_robot_description/urdf/robot_arm.urdf (robot description, URDF)
Before this commit: robot koch_v11_writing_arm, 7 links, 6 joints
Joints:
- joint elbow_flex: axis 0.000000 1.000000 0.000000 -> 0.000000 -1.000000 0.000000; origin xyz=0.109000 0.000000 -0.014000 rpy=0.000000 0.000000 0.000000 -> xyz=0.109000 0.000000 -0.013000 rpy=3.14159 0.000000 0.000000
- joint pen_holder: origin xyz=0.000000 -0.007000 0.015000 rpy=0.000000 0.000000 0.000000 -> xyz=0.000000 -0.007000 0.016000 rpy=0.785398 0.000000 0.000000
- joint shoulder_lift: origin xyz=-0.001000 0.000000 0.038000 rpy=0.000000 0.000000 0.000000 -> xyz=-0.001000 0.000000 0.038000 rpy=3.14159  0.000000 0.000000
- joint shoulder_pan: axis 0.000000 0.000000 1.000000 -> 0.000000 0.000000 -1.000000; origin xyz=0.001000 0.000000 0.021000 rpy=0.000000 0.000000 0.000000 -> xyz=0.001000 0.017000 0.042000 rpy=0.000000 0.000000 0.000000
- joint wrist_flex: origin xyz=0.101000 0.000000 0.002000 rpy=0.000000 0.000000 0.000000 -> xyz=0.101000 -0.001000 0.003000 rpy=0.000000 0.000000 0.000000
- joint wrist_roll: origin xyz=-0.001000 0.000000 0.039000 rpy=0.000000 0.000000 0.000000 -> xyz=-0.001000 0.001000 0.043000 rpy=0.000000 0.000000 0.000000
