Commit message: initial STL setup for RVIZ

File: writing_robot_description/urdf/koch_v11_arm_real.urdf (robot description, URDF)
Before this commit: robot koch_v11_writing_arm, 8 links, 7 joints
Links:
- link base_link: geometry collision cylinder length=0.02 radius=0.05; visual mesh filename=package://writing_robot_description/meshes/Follower_Base.STL
- link shoulder_link: geometry visual mesh filename=package://writing_robot_description/meshes/XL-430_new.stl scale=0.001 0.001 0.001; visual mesh filename=package://writing_robot_description/meshes/fr12_s102.stl scale=0.001 0.001 0.001

Commit message: STL binary conversion as needed by RVIZ

File: writing_robot_description/urdf/koch_v11_arm_real.urdf (robot description, URDF)
Before this commit: robot koch_v11_writing_arm, 8 links, 7 joints
Links:
- link base_link: geometry collision cylinder length=0.02 radius=0.05; visual mesh filename=package://writing_robot_description/meshes/Follower_Base_bi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

Commit message: add rest of binary stls for the attachments

File: writing_robot_description/urdf/koch_v11_arm_real.urdf (robot description, URDF)
Before this commit: robot koch_v11_writing_arm, 8 links, 7 joints
Links:
- link base_link: geometry collision cylinder length=0.02 radius=0.05; visual mesh filename=package://writing_robot_description/meshes/Follower_Base_bi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 scale=0.001 0.001 0.001
- link upper_arm_link: geometry visual mesh filename=package://writing_robot_description/meshes/Follower_Shoulde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 scale=0.001 0.001 0.001; visual mesh filename=package://writing_robot_description/meshes/XL,XC-330.stl scale=0.001 0.001 0.001
Joints:
- joint shoulder_pan: origin xyz=0 0 0.02 rpy=0 0 0 -> xyz=0 0 0.04 rpy=0 0 0

Commit message: fix mesh path issue

File: writing_robot_description/urdf/koch_v11_arm_real.urdf (robot description, URDF)
Before this commit: robot koch_v11_writing_arm, 8 links, 7 joints
Links:
- link forearm_link: geometry visual mesh filename=package://writing_robot_description/meshes/Follower_Elbow_T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 scale=0.001 0.001 0.001; visual mesh filename=package://writing_robot_description/meshes/XL,XC-330.stl scale=0.001 0.001 0.001
- link hand_link: geometry visual mesh filename=package://writing_robot_description/meshes/Follower_Elbow_T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 scale=0.001 0.001 0.001; visual mesh filename=package://writing_robot_description/meshes/XL,XC-330.stl scale=0.001 0.001 0.001
- link pen_link: geometry visual mesh filename=package://writing_robot_description/meshes/Follower_Gripper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 scale=0.001 0.001 0.001; visual mesh filename=package://writing_robot_description/meshes/XL,XC-330.stl scale=0.001 0.001 0.001
- link wrist_link: geometry visual mesh filename=package://writing_robot_description/meshes/Follower_Elbow_T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 scale=0.001 0.001 0.001; visual mesh filename=package://writing_robot_description/meshes/XL,XC-330.stl scale=0.001 0.001 0.001

Commit message: relfecting extraction fix

File: writing_robot_description/urdf/koch_v11_arm_real.urdf (robot description, URDF)
Before this commit: robot koch_v11_writing_arm, 8 links, 7 joints
Joints:
- joint elbow_flex: axis 0.000000 -1.000000 -0.000000 -> 0.000000 0.000000 1.000000; origin xyz=0.002000 -0.014000 -0.100000 rpy=-0.000000 0.000000 -3.141593 -> xyz=0.002000 0.100000 -0.014000 rpy=-0.000000 0.000000 -3.141593
- joint pen_holder: axis 0.000000 -1.000000 0.000000 -> 0.000000 0.000000 1.000000; origin xyz=-0.213000 0.008000 -0.055000 rpy=3.141593 0.000000 1.570796 -> xyz=-0.055000 0.008000 0.213000 rpy=3.141593 0.000000 1.570796
- joint shoulder_lift: axis 0.000000 1.000000 -0.000000 -> 0.000000 0.000000 1.000000; origin xyz=0.109000 0.009000 -0.014000 rpy=3.141593 0.000000 0.000000 -> xyz=0.109000 -0.014000 -0.009000 rpy=3.141593 0.000000 0.000000
- joint shoulder_pan: axis 0.000000 -1.000000 0.000000 -> 0.000000 0.000000 1.000000
- joint wrist_flex: axis 0.000000 0.000000 -1.000000 -> 0.000000 0.000000 1.000000; origin xyz=0.000000 0.021000 -0.038000 rpy=1.570796 -0.000000 0.000000 -> xyz=0.000000 0.038000 -0.021000 rpy=1.570796 -0.000000 0.000000
- joint wrist_roll: axis -1.000000 0.000000 -0.000000 -> 0.000000 0.000000 1.000000; origin xyz=-0.008000 0.009000 -0.019000 rpy=0.000000 1.570796 0.000000 -> xyz=0.008000 0.009000 0.019000 rpy=0.000000 1.570796 0.000000

Commit message: additional fixes

File: writing_robot_description/urdf/koch_v11_arm_real.urdf (robot description, URDF)
Before this commit: robot koch_v11_writing_arm, 8 links, 7 joints
Joints:
- joint elbow_flex: axis 0.000000 0.000000 1.000000 -> 0.000000 -1.000000 0.000000
- joint shoulder_lift: axis 0.000000 0.000000 1.000000 -> 0.000000 1.000000 0.000000
- joint shoulder_pan: axis 0.000000 0.000000 1.000000 -> 0.000000 1.000000 0.000000
- joint wrist_flex: axis 0.000000 0.000000 1.000000 -> 0.000000 0.000000 -1.000000
- joint wrist_roll: axis 0.000000 0.000000 1.000000 -> -1.000000 0.000000 0.000000

Commit message: reflect display changes to the real robot urdf

File: writing_robot_description/urdf/koch_v11_arm_real.urdf (robot description, URDF)
Before this commit: robot koch_v11_writing_arm, 8 links, 7 joints
Links:
- removed link pen_tip
- link hand_link: geometry visual mesh filename=package://writing_robot_description/meshes/Follower_Gripper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 scale=0.001 0.001 0.001; visual mesh filename=package://writing_robot_description/meshes/XL,XC-330.stl scale=0.001 0.001 0.001
- link pen_link: geometry visual mesh filename=package://writing_robot_description/meshes/Follower_Gripper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 scale=0.001 0.001 0.001
Joints:
- removed joint pen_tip_joint
- joint elbow_flex: axis 0.000000 -1.000000 0.000000 -> 1.000000 0.000000 0.000000; origin xyz=0.002000 0.100000 -0.014000 rpy=-0.000000 0.000000 -3.141593 -> xyz=-0.000000 -0.108000 0.014000 rpy=0.000000 -0.000000 -0.000000
- joint pen_holder: axis 0.000000 0.000000 1.000000 -> 0.000000 1.000000 0.000000; origin xyz=-0.055000 0.008000 0.213000 rpy=3.141593 0.000000 1.570796 -> xyz=0.000000 -0.009000 0.015000 rpy=0.000000 -0.000000 -1.570796
- joint shoulder_lift: axis 0.000000 1.000000 0.000000 -> 1.000000 0.000000 0.000000; origin xyz=0.109000 -0.014000 -0.009000 rpy=3.141593 0.000000 0.000000 -> xyz=0.000000 0.002000 -0.001000 rpy=1.570796 1.570796 -1.570796
- joint shoulder_pan: axis 0.000000 1.000000 0.000000 -> 0.000000 -1.000000 0.000000
- joint wrist_flex: axis 0.000000 0.000000 -1.000000 -> -1.000000 0.000000 0.000000; origin xyz=0.000000 0.038000 -0.021000 rpy=1.570796 -0.000000 0.000000 -> xyz=-0.001000 -0.100000 0.002000 rpy=0.000000 -0.000000 -0.000000
- joint wrist_roll: axis -1.000000 0.000000 0.000000 -> 0.000000 0.000000 1.000000; origin xyz=0.008000 0.009000 0.019000 rpy=0.000000 1.570796 0.000000 -> xyz=0.003000 -0.001000 -0.044000 rpy=3.141593 -0.000000 -1.570796

Commit message: intermediate change

File: writing_robot_description/urdf/koch_v11_arm_real.urdf (robot description, URDF)
Before this commit: robot koch_v11_writing_arm, 7 links, 6 joints
Joints:
- joint shoulder_lift: axis 1.000000 0.000000 0.000000 -> -1.000000 0.000000 0.000000

Commit message: reflecting fix into real robot urdf

File: writing_robot_description/urdf/koch_v11_arm_real.urdf (robot description, URDF)
Before this commit: robot koch_v11_writing_arm, 7 links, 6 joints
Joints:
- joint elbow_flex: axis 1.000000 0.000000 0.000000 -> 0.000000 1.000000 0.000000; origin xyz=-0.000000 -0.108000 0.014000 rpy=0.000000 -0.000000 -0.000000 -> xyz=0.109000 0.000000 -0.014000 rpy=0.000000 0.000000 0.000000
- joint pen_holder: axis 0.000000 1.000000 0.000000 -> -1.000000 0.000000 0.000000; origin xyz=0.000000 -0.009000 0.015000 rpy=0.000000 -0.000000 -1.570796 -> xyz=0.000000 -0.007000 0.015000 rpy=0.000000 0.000000 0.000000
- joint shoulder_lift: axis -1.000000 0.000000 0.000000 -> 0.000000 1.000000 0.000000; origin xyz=0.000000 0.002000 -0.001000 rpy=1.570796 1.570796 -1.570796 -> xyz=-0.001000 0.000000 0.038000 rpy=0.000000 0.000000 0.000000
- joint shoulder_pan: axis 0.000000 -1.000000 0.000000 -> 0.000000 0.000000 1.000000; origin xyz=0.000000 0.000000 0.059000 rpy=1.570796 0.000000 0.000000 -> xyz=0.001000 0.000000 0.021000 rpy=0.000000 0.000000 0.000000
- joint wrist_flex: axis -1.000000 0.000000 0.000000 -> 0.000000 1.000000 0.000000; origin xyz=-0.001000 -0.100000 0.002000 rpy=0.000000 -0.000000 -0.000000 -> xyz=0.101000 0.000000 0.002000 rpy=0.000000 0.000000 0.000000
- joint wrist_roll: origin xyz=0.003000 -0.001000 -0.044000 rpy=3.141593 -0.000000 -1.570796 -> xyz=-0.001000 0.000000 0.039000 rpy=0.000000 0.000000 0.000000

Commit message: adjustments to two joint angles

File: writing_robot_description/urdf/koch_v11_arm_real.urdf (robot description, URDF)
Before this commit: robot koch_v11_writing_arm, 7 links, 6 joints
Joints:
- joint elbow_flex: origin xyz=0.109000 0.000000 -0.014000 rpy=0.000000 0.000000 0.000000 -> xyz=0.109000 0.000000 -0.014000 rpy=3.14159 0.000000 0.000000
- joint shoulder_lift: origin xyz=-0.001000 0.000000 0.038000 rpy=0.000000 0.000000 0.000000 -> xyz=-0.001000 0.000000 0.038000 rpy=3.14159  0.000000 0.000000
- joint shoulder_pan: axis 0.000000 0.000000 1.000000 -> 0.000000 0.000000 -1.000000

Commit message: fixed thumb overreach

File: writing_robot_description/urdf/koch_v11_arm_real.urdf (robot description, URDF)
Before this commit: robot koch_v11_writing_arm, 7 links, 6 joints
Joints:
- joint pen_holder: origin xyz=0.000000 -0.007000 0.015000 rpy=0.000000 0.000000 0.000000 -> xyz=0.000000 -0.007000 0.015000 rpy=0.785398 0.000000 0.000000

Commit message: pose test program to validate poses

File: writing_robot_description/urdf/koch_v11_arm_real.urdf (robot description, URDF)
Before this commit: robot koch_v11_writing_arm, 7 links, 6 joints
Joints:
- joint elbow_flex: origin xyz=0.109000 0.000000 -0.014000 rpy=3.14159 0.000000 0.000000 -> xyz=0.109000 0.000000 -0.013000 rpy=3.14159 0.000000 0.000000
- joint pen_holder: origin xyz=0.000000 -0.007000 0.015000 rpy=0.785398 0.000000 0.000000 -> xyz=0.000000 -0.007000 0.016000 rpy=0.785398 0.000000 0.000000
- joint shoulder_pan: origin xyz=0.001000 0.000000 0.021000 rpy=0.000000 0.000000 0.000000 -> xyz=0.001000 0.017000 0.042000 rpy=0.000000 0.000000 0.000000
- joint wrist_flex: origin xyz=0.101000 0.000000 0.002000 rpy=0.000000 0.000000 0.000000 -> xyz=0.101000 -0.001000 0.003000 rpy=0.000000 0.000000 0.000000
- joint wrist_roll: origin xyz=-0.001000 0.000000 0.039000 rpy=0.000000 0.000000 0.000000 -> xyz=-0.001000 0.001000 0.043000 rpy=0.000000 0.000000 0.000000

Commit message: cleaned up transmission matrix for joint 3

File: writing_robot_description/urdf/koch_v11_arm_real.urdf (robot description, URDF)
Before this commit: robot koch_v11_writing_arm, 7 links, 6 joints
Joints:
- joint elbow_flex: axis 0.000000 1.000000 0.000000 -> 0.000000 -1.000000 0.000000

Commit message: fix for base joint 1 rotating the wrong direction in rviz

File: writing_robot_description/urdf/koch_v11_arm_real.urdf (robot description, URDF)
Before this commit: robot koch_v11_writing_arm, 7 links, 6 joints
Joints:
- joint shoulder_pan: axis 0.000000 0.000000 -1.000000 -> 0.000000 0.000000 1.000000

Commit message: fix for wrist roll being off by 90 degrees in rviz from real robot

File: writing_robot_description/urdf/koch_v11_arm_real.urdf (robot description, URDF)
Before this commit: robot koch_v11_writing_arm, 7 links, 6 joints
Joints:
- joint wrist_roll: origin xyz=-0.001000 0.001000 0.043000 rpy=0.000000 0.000000 0.000000 -> xyz=-0.001000 0.001000 0.043000 rpy=0.000000 0.000000 1.570796

Commit message: one more tweak to that fix

File: writing_robot_description/urdf/koch_v11_arm_real.urdf (robot description, URDF)
Before this commit: robot koch_v11_writing_arm, 7 links, 6 joints
Joints:
- joint wrist_roll: origin xyz=-0.001000 0.001000 0.043000 rpy=0.000000 0.000000 1.570796 -> xyz=-0.001000 0.001000 0.043000 rpy=0.000000 0.000000 -1.570796

Commit message: fix for wrong angle for shoulder lift

File: writing_robot_description/urdf/koch_v11_arm_real.urdf (robot description, URDF)
Before this commit: robot koch_v11_writing_arm, 7 links, 6 joints
Joints:
- joint shoulder_lift: axis 0.000000 1.000000 0.000000 -> 0.000000 -1.000000 0.000000; origin xyz=-0.001000 0.000000 0.038000 rpy=3.14159  0.000000 0.000000 -> xyz=-0.001000 0.000000 0.038000 rpy=3.14159  1.570796 0.000000

Commit message: calculations and additions to urdf for inertial properties

File: writing_robot_description/urdf/koch_v11_arm_real.urdf (robot description, URDF)
Before this commit: robot koch_v11_writing_arm, 7 links, 6 joints
Links:
- link base_link: mass 0.5 -> 0.089861
- link forearm_link: mass 0.15 -> 0.088473
- link hand_link: mass 0.08 -> 0.045639
- link pen_link: mass 0.02 -> 0.015925
- link shoulder_link: mass 0.3 -> 0.061576
- link upper_arm_link: mass 0.2 -> 0.071602
- link wrist_link: mass 0.1 -> 0.034634

Commit message: collision update in urdf

File: writing_robot_description/urdf/koch_v11_arm_real.urdf (robot description, URDF)
Before this commit: robot koch_v11_writing_arm, 7 links, 6 joints
Links:
- link forearm_link: geometry collision box size=0.045000 0.100086 0.033000; collision cylinder length=0.028000 radius=0.017000
- link hand_link: geometry collision cylinder length=0.028000 radius=0.017000; collision cylinder length=0.078868 radius=0.021813
- link pen_link: geometry collision box size=0.073917 0.045500 0.031000; visual mesh filename=package://writing_robot_description/meshes/Follower_Gripper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 scale=0.001 0.001 0.001
- link shoulder_link: geometry collision box size=0.047000 0.038000 0.021500; collision cylinder length=0.046000 radius=0.019000
- link upper_arm_link: geometry collision box size=0.054000 0.141912 0.036000; collision cylinder length=0.028000 radius=0.017000
- link wrist_link: geometry collision cylinder length=0.028000 radius=0.017000; collision cylinder length=0.052000 radius=0.017487

Commit message: load testing tool and pose_test improvements

File: writing_robot_description/urdf/koch_v11_arm_real.urdf (robot description, URDF)
Before this commit: robot koch_v11_writing_arm, 7 links, 6 joints
Joints:
- joint elbow_flex: limit lower=-2.5 upper=2.5 effort=1.5 velocity=3.14 -> lower=0.926 upper=1.650 effort=1.5 velocity=3.14
- joint pen_holder: limit lower=-0.5 upper=0.5 effort=0.5 velocity=1.57 -> lower=1.60 upper=0.19 effort=0.5 velocity=1.57
- joint shoulder_lift: limit lower=-2.0 upper=2.0 effort=2.0 velocity=3.14 -> lower=2.8857 upper=2.486 effort=2.0 velocity=3.14
- joint shoulder_pan: limit lower=-3.14159 upper=3.14159 effort=2.0 velocity=3.14 -> lower=2.044 upper=0.540 effort=2.0 velocity=3.14
- joint wrist_flex: limit lower=-2.0 upper=2.0 effort=1.5 velocity=3.14 -> lower=2.70 upper=0.297 effort=1.5 velocity=3.14
- joint wrist_roll: limit lower=-3.14159 upper=3.14159 effort=1.0 velocity=3.14 -> lower=1.448 upper=-1.448 effort=1.0 velocity=3.14

Commit message: some bug fixes and addition of new delivery pose set v1.0

File: writing_robot_description/urdf/koch_v11_arm_real.urdf (robot description, URDF)
Before this commit: robot koch_v11_writing_arm, 7 links, 6 joints
Joints:
- joint elbow_flex: limit lower=0.926 upper=1.650 effort=1.5 velocity=3.14 -> lower=0.726 upper=2.250 effort=1.5 velocity=3.14
- joint shoulder_lift: limit lower=2.8857 upper=2.486 effort=2.0 velocity=3.14 -> lower=2.8857 upper=2.2000 effort=2.0 velocity=3.14
- joint wrist_roll: limit lower=1.448 upper=-1.448 effort=1.0 velocity=3.14 -> lower=1.900 upper=-1.448 effort=1.0 velocity=3.14
