Commit message: urdf update for balance exercise

File: writing_robot_description/urdf/koch_v11_arm_real_for_balance.urdf (robot description, URDF)
Before this commit: robot koch_v11_writing_arm, 7 links, 6 joints
Links:
- added link ball_link, mass 0.014; collision sphere radius=0.0075; visual sphere radius=0.0075
- added link cup_plate_link, mass 0.050; collision cylinder length=0.008 radius=0.060; visual cylinder length=0.008 radius=0.030
- added link cup_ring_link, mass 0.030; collision cylinder length=0.045 radius=0.035; visual cylinder length=0.045 radius=0.015
Joints:
- added joint ball_joint: type fixed, parent cup_ring_link, child ball_link, origin xyz=0.0 0.0 -0.04 rpy=0 0 0
- added joint cup_plate_joint: type fixed, parent pen_link, child cup_plate_link, origin xyz=0.03 0.00 0.04 rpy=3.1416 1.5708 0
- added joint cup_ring_joint: type fixed, parent cup_plate_link, child cup_ring_link, origin xyz=0.000 0.0 0.03 rpy=0 0 0

Commit message: tune the model to reflect right order

File: writing_robot_description/urdf/koch_v11_arm_real_for_balance.urdf (robot description, URDF)
Before this commit: robot koch_v11_writing_arm, 10 links, 9 joints
Links:
- removed link cup_ring_link
- added link cup_handle_link, mass 0.030; collision cylinder length=0.045 radius=0.015; visual cylinder length=0.035 radius=0.015
Joints:
- removed joint cup_ring_joint
- added joint cup_handle_joint: type fixed, parent pen_link, child cup_handle_link, origin xyz=0.00 0.00 0.04 rpy=0 1.5708 0
- joint ball_joint: origin xyz=0.0 0.0 -0.04 rpy=0 0 0 -> xyz=0.0 0.0 0.0115 rpy=0 0 0; parent cup_ring_link -> cup_plate_link
- joint cup_plate_joint: origin xyz=0.03 0.00 0.04 rpy=3.1416 1.5708 0 -> xyz=0.0 0.0 0.02 rpy=0 0 0; parent pen_link -> cup_handle_link

Commit message: unified pid on vision and imu plus other tuning of urdf

File: writing_robot_description/urdf/koch_v11_arm_real_for_balance.urdf (robot description, URDF)
Before this commit: robot koch_v11_writing_arm, 10 links, 9 joints
Links:
- removed link ball_link
Joints:
- removed joint ball_joint
