Commit message: pen_holder to gripper

File: robot_arm_description/urdf/koch_v11_arm_real.urdf (robot description, URDF)
Before this commit: robot koch_v11_writing_arm, 7 links, 6 joints
Joints:
- removed joint pen_holder
- added joint gripper: type revolute, parent hand_link, child gripper, origin xyz=0.000000 -0.007000 0.016000 rpy=0.785398 0.000000 0.000000, axis -1.000000 0.000000 0.000000, limit lower=1.60 upper=0.19 effort=0.5 velocity=1.57

File: robot_arm_description/urdf/koch_v11_arm_real_for_balance.urdf (robot description, URDF)
Before this commit: robot koch_v11_writing_arm, 9 links, 8 joints
Joints:
- removed joint pen_holder
- added joint gripper: type revolute, parent hand_link, child gripper, origin xyz=0.000000 -0.007000 0.016000 rpy=0.785398 0.000000 0.000000, axis -1.000000 0.000000 0.000000, limit lower=1.60 upper=0.19 effort=0.5 velocity=1.57

File: robot_arm_description/urdf/koch_v11_arm_simple_sim.urdf (robot description, URDF)
Before this commit: robot koch_v11_writing_arm, 8 links, 7 joints
Joints:
- removed joint pen_holder
- added joint gripper: type revolute, parent hand_link, child gripper, origin xyz=0.10 0 0 rpy=0 0 0, axis 0 1 0, limit lower=-0.5 upper=0.5 effort=0.5 velocity=1.57
