Commit message: updates to urdf and related files to support rviz simulation

File: robot_arm_description/urdf/so_arm101.urdf (robot description, URDF)
Before this commit: robot so_101_arm, 7 links, 6 joints
Links:
- removed link link1
- removed link link2
- removed link link3
- removed link link4
- removed link link5
- removed link link6
- added link gripper_frame_link, mass 1e-9
- added link gripper_link, mass 0.087; collision mesh filename=package://robot_arm_description/meshes/so101/sts3215_03a_v1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; collision mesh filename=package://robot_arm_description/meshes/so101/wrist_roll_fol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
- added link lower_arm_link, mass 0.104; collision mesh filename=package://robot_arm_description/meshes/so101/motor_holder_s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; collision mesh filename=package://robot_arm_description/meshes/so101/sts3215_03a_v1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
- added link moving_jaw_so101_v1_link, mass 0.012; collision mesh filename=package://robot_arm_description/meshes/so101/moving_jaw_so1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; visual mesh filename=package://robot_arm_description/meshes/so101/moving_jaw_so1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
- added link shoulder_link, mass 0.100006; collision mesh filename=package://robot_arm_description/meshes/so101/motor_holder_s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; collision mesh filename=package://robot_arm_description/meshes/so101/rotation_pitch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
- added link upper_arm_link, mass 0.103; collision mesh filename=package://robot_arm_description/meshes/so101/sts3215_03a_v1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; collision mesh filename=package://robot_arm_description/meshes/so101/upper_arm_so10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
- added link wrist_link, mass 0.079; collision mesh filename=package://robot_arm_description/meshes/so101/sts3215_03a_no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; collision mesh filename=package://robot_arm_description/meshes/so101/wrist_roll_pit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
- link base_link: mass None -> 0.147; geometry collision mesh filename=package://robot_arm_description/meshes/so101/base_motor_hol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; collision mesh filename=package://robot_arm_description/meshes/so101/base_so101_v2.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
Joints:
- added joint gripper_frame_joint: type fixed, parent gripper_link, child gripper_frame_link, origin xyz=-0.0079 -0.000218121 -0.0981274 rpy=0 3.14159 0, axis 0 0 0
- joint elbow_flex: axis 0 1 0 -> 0 0 1; child link3 -> lower_arm_link; limit lower=-1.69 upper=1.69 effort=4.5 velocity=6.0 -> lower=-1.69 upper=1.69 effort=10 velocity=10; origin xyz=0 0 0.10 rpy=0 0 0 -> xyz=-0.11257 -0.028 1.73763e-16 rpy=-3.63608e-16 8.74301e-16 1.5708; parent link2 -> upper_arm_link
- joint gripper: axis 0 1 0 -> 0 0 1; child link6 -> moving_jaw_so101_v1_link; limit lower=-1.0 upper=1.0 effort=4.5 velocity=6.0 -> lower=-0.174533 upper=1.74533 effort=10 velocity=10; origin xyz=0 0 0.03 rpy=0 0 0 -> xyz=0.0202 0.0188 -0.0234 rpy=1.5708 -5.24284e-08 -1.41553e-15; parent link5 -> gripper_link
- joint shoulder_lift: axis 0 -1 0 -> 0 0 1; child link2 -> upper_arm_link; limit lower=-1.74 upper=1.74 effort=4.5 velocity=6.0 -> lower=-1.74533 upper=1.74533 effort=10 velocity=10; origin xyz=0 0 0.05 rpy=0 0 0 -> xyz=-0.0303992 -0.0182778 -0.0542 rpy=-1.5708 -1.5708 0; parent link1 -> shoulder_link
- joint shoulder_pan: child link1 -> shoulder_link; limit lower=-3.14 upper=3.14 effort=4.5 velocity=6.0 -> lower=-1.91986 upper=1.91986 effort=10 velocity=10; origin xyz=0 0 0.05 rpy=0 0 0 -> xyz=0.0388353 -8.97657e-09 0.0624 rpy=3.14159 4.18253e-17 -3.14159
- joint wrist_flex: axis 0 1 0 -> 0 0 1; child link4 -> wrist_link; limit lower=-1.65 upper=1.65 effort=4.5 velocity=6.0 -> lower=-1.65806 upper=1.65806 effort=10 velocity=10; origin xyz=0 0 0.10 rpy=0 0 0 -> xyz=-0.1349 0.0052 3.62355e-17 rpy=4.02456e-15 8.67362e-16 -1.5708; parent link3 -> lower_arm_link
- joint wrist_roll: axis -1 0 0 -> 0 0 1; child link5 -> gripper_link; limit lower=-3.14 upper=3.14 effort=4.5 velocity=6.0 -> lower=-2.74385 upper=2.84121 effort=10 velocity=10; origin xyz=0 0 0.05 rpy=0 0 0 -> xyz=5.55112e-17 -0.0611 0.0181 rpy=1.5708 0.0486795 3.14159; parent link4 -> wrist_link
