Commit message: adjustments to show the cup being held by the gripper

File: robot_arm_description/urdf/so_arm101_for_balance.urdf (robot description, URDF)
Before this commit: robot so_arm101_for_balance, 10 links, 9 joints
Joints:
- joint cup_handle_joint: origin xyz=0 0 0.0175 rpy=0 0 0 -> xyz=-0.01 -0.0175 -0.02 rpy=1.5708 0 0

Commit message: fix to render ball movement correctly

File: robot_arm_description/urdf/so_arm101_for_balance.urdf (robot description, URDF)
Before this commit: robot so_arm101_for_balance, 10 links, 9 joints
Joints:
- joint cup_plate_joint: origin xyz=0 0 0.02 rpy=0 0 0 -> xyz=0 0 0.02 rpy=0 0 1.5708

Commit message: fix to render ball movement correctly ... one more fix

File: robot_arm_description/urdf/so_arm101_for_balance.urdf (robot description, URDF)
Before this commit: robot so_arm101_for_balance, 10 links, 9 joints
Joints:
- joint cup_plate_joint: origin xyz=0 0 0.02 rpy=0 0 1.5708 -> xyz=0 0 0.02 rpy=0 0 -1.5708
